Commit message: Initial vreation

File: src/bumperbot_description/urdf/bumperbot_gazebo.xacro (robot description, xacro)
@@ -1,4 +1,5 @@
 <?xml version="1.0"?>
 <robot name="bumperbot" xmlns:xacro="http://www.ros.org/wiki/xacro">
+    <!-- -->
     <transmission name="wheel_right_transmission">
         <plugin>trannsmission_interface/SimpleTransmission</plugin>
@@ -8,4 +9,5 @@
         </joint>
     </transmission>
+    <!-- -->
     <transmission name="wheel_left_transmission">
         <plugin>trannsmission_interface/SimpleTransmission</plugin>
@@ -51,8 +53,57 @@
     <gazebo>
         <plugin filename="libgazebo_ros2_control.so" name="gazebo_ros2_control">
-            <robot_param>robot_dexcription</robot_param>
+            <robot_param>robot_description</robot_param>
             <robot_param_node>robot_state_publisher</robot_param_node>
-            <parameters>$(find bumperbot_controller)/share/config/bumperbot_controllers.yaml</parameters>
+            <parameters>$(find bumperbot_controller)/config/bumperbot_controllers.yaml</parameters>
         </plugin>
     </gazebo>
+    <gazebo reference="imu_link">
+        <sensor name="imu" type="imu">
+            <always_on>true</always_on>
+            <update_rate>100</update_rate>
+            <imu>
+                <angular_velocity>
+                    <x>
+                        <noise type="gaussian">
+                            <mean>0.0</mean>
+                            <stddev>2e-4</stddev>
+                        </noise>
+                    </x>
+                    <y>
+                        <noise type="gaussian">
+                            <mean>0.0</mean>
+                            <stddev>2e-4</stddev>
+                        </noise>
+                    </y>
+                    <z>
+                        <noise type="gaussian">
+                            <mean>0.0</mean>
+                            <stddev>2e-4</stddev>
+                        </noise>
+                    </z>
+                </angular_velocity>
+                <linear_acceleration>
+                    <x>
+                        <noise type="gaussian">
+                            <mean>0.0</mean>
+                            <stddev>1.7e-2</stddev>
+                        </noise>
+                    </x>
+                    <y>
+                        <noise type="gaussian">
+                            <mean>0.0</mean>
+                            <stddev>1.7e-2</stddev>
+                        </noise>
+                    </y>
+                    <z>
+                        <noise type="gaussian">
+                            <mean>0.0</mean>
+                            <stddev>1.7e-2</stddev>
+                        </noise>
+                    </z>
+                </linear_acceleration>
+            </imu>
+            <plugin name="imu" filename="libgazebo_ros_imu_sensor.so"/>
+        </sensor>
+    </gazebo>
 </robot>

File: src/bumperbot_description/urdf/bumperbot_ros2_control.xacro (robot description, xacro)
@@ -2,7 +2,15 @@
 <robot name="bumperbot" xmlns:xacro="http://www.ros.org/wiki/xacro">
     <ros2_control type="system" name="RobotSystem">
-        <hardware>
-            <plugin>gazebo_ros2_control/GazeboSystem</plugin>
-        </hardware>
+        <xacro:if value="$(arg is_sim)">
+            <hardware>
+                <plugin>gazebo_ros2_control/GazeboSystem</plugin>
+            </hardware>
+        </xacro:if>
+        <xacro:unless value="$(arg is_sim)">
+            <hardware>
+                <plugin>bumperbot_firmware/BumperbotInterface</plugin>
+                <param name="port">/dev/ttyUSB0</param>
+            </hardware>
+        </xacro:unless>
         <joint name="wheel_right_joint">
             <command_interface name="velocity">

File: src/bumperbot_description/urdf/bumperbot_urdf.xacro (robot description, xacro)
@@ -1,4 +1,5 @@
 <?xml version="1.0"?>
 <robot name="bumperbot" xmlns:xacro="http://www.ros.org/wiki/xacro">
+    <xacro:arg name="is_sim" default="true"/>
     <!-- Include other URDF files-->
     <xacro:include filename="$(find bumperbot_description)/urdf/bumperbot_gazebo.xacro"/>
@@ -143,4 +144,30 @@
         <origin xyz="-0.04755 0 -0.0275" rpy="0 0 0"/>
     </joint>
+    <link name="imu_link">
+        <inertial>
+            <origin xyz="-0.00552433659106688 0.000168210391520346 0.000514000497342681" rpy="0 0 0" />
+            <mass value="0.000528415362211671" />
+            <inertia ixx="1.46176048428261E-08" ixy="1.40015117949421E-10" ixz="-1.99633872937403E-12"
+                     iyy="8.59662482954888E-09" iyz="7.52375112767959E-12"
+                     izz="2.30279421279312E-08" />
+        </inertial>
+        <visual>
+            <origin xyz="0 0 0" rpy="0 0 0"/>
+            <geometry>
+                <mesh filename="package://bumperbot_description/meshes/imu_link.STL"/>
+            </geometry>
+        </visual>
+        <collision>
+            <origin xyz="0 0 0" rpy="0 0 0"/>
+            <geometry>
+                <mesh filename="package://bumperbot_description/meshes/imu_link.STL"/>
+            </geometry>
+        </collision>
+    </link>
+    <joint name="imu_joint" type="fixed">
+        <parent link="base_link"/>
+        <child link="imu_link"/>
+        <origin xyz="0 0 0.07" rpy="0 0 0"/>
+    </joint>
     <!-- Can -->
     <!-- <link name="can_link">
